File: PCB/Ducker-Charger/Ducker-Charger.kicad_sch (KiCad schematic)
At the start: 2 parts, among them J1 Conn_01x02, J2 Conn_01x05

Commit message: fix: I2C is now a BUS, no longer a global label
Other:
- sheet BMS ports: added I2C_LP{I2C}; removed none
- sheet High_pow ports: added I2C_PD{I2C}; removed none
- sheet Logic ports: added I2C_LP{I2C}, I2C_PD{I2C}; removed none
- sheet Low_pow ports: added I2C_LP{I2C}; removed none
Changed lines of the file:
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@@
 	(text "LOW POWER\n"
 		(exclude_from_sim no)
-		(at 248.666 90.678 0)
+		(at 248.666 48.768 0)
 		(effects
 			(font
@@
 	(text "HIGH POWER\n"
 		(exclude_from_sim no)
-		(at 248.92 50.546 0)
+		(at 248.92 92.71 0)
 		(effects
 			(font
@@
 		)
 	)
+	(junction
+		(at 219.71 123.19)
+		(diameter 0)
+		(color 0 0 0 0)
+	)
 	(wire
 		(pts
@@
 		)
 	)
+	(bus
+		(pts
+			(xy 219.71 64.77) (xy 227.33 64.77)
+		)
+		(stroke
+			(width 0)
+			(type default)
+		)
+	)
+	(bus
+		(pts
+			(xy 224.79 119.38) (xy 224.79 106.68)
+		)
+		(stroke
+			(width 0)
+			(type default)
+		)
+	)
 	(wire
 		(pts
@@
 		)
 	)
+	(bus
+		(pts
+			(xy 182.88 123.19) (xy 219.71 123.19)
+		)
+		(stroke
+			(width 0)
+			(type default)
+		)
+	)
+	(bus
+		(pts
+			(xy 219.71 123.19) (xy 219.71 64.77)
+		)
+		(stroke
+			(width 0)
+			(type default)
+		)
+	)
+	(bus
+		(pts
+			(xy 224.79 106.68) (xy 227.33 106.68)
+		)
+		(stroke
+			(width 0)
+			(type default)
+		)
+	)
+	(bus
+		(pts
+			(xy 227.33 123.19) (xy 219.71 123.19)
+		)
+		(stroke
+			(width 0)
+			(type default)
+		)
+	)
 	(wire
 		(pts
 			(xy 39.37 71.12) (xy 39.37 76.2)
+		)
+		(stroke
+			(width 0)
+			(type default)
+		)
+	)
+	(bus
+		(pts
+			(xy 227.33 119.38) (xy 224.79 119.38)
 		)
 		(stroke
@@
 	)
 	(sheet
-		(at 106.045 71.12)
-		(size 76.2 55.245)
+		(at 106.68 71.12)
+		(size 76.2 55.88)
 		(exclude_from_sim no)
 		(in_bom yes)
@@
 		)
 		(property "Sheetname" "BMS"
-			(at 106.045 70.4084 0)
+			(at 106.68 70.4084 0)
 			(effects
 				(font
@@
 		)
 		(property "Sheetfile" "BMS.kicad_sch"
-			(at 106.045 126.9496 0)
+			(at 106.68 126.9496 0)
 			(effects
 				(font
@@
 				)
 				(justify left top)
+			)
+		)
+		(pin "I2C_LP{I2C}" bidirectional
+			(at 182.88 123.19 0)
+			(effects
+				(font
+					(size 1.27 1.27)
+				)
+				(justify right)
 			)
 		)
@@
 	)
 	(sheet
-		(at 227.33 72.39)
+		(at 227.33 30.48)
 		(size 43.815 37.465)
 		(exclude_from_sim no)
@@
 		)
 		(property "Sheetname" "Low_pow"
-			(at 227.33 71.6784 0)
+			(at 227.33 29.7684 0)
 			(effects
 				(font
@@
 		)
 		(property "Sheetfile" "low_pow.kicad_sch"
-			(at 227.33 110.4396 0)
+			(at 227.33 68.5296 0)
 			(effects
 				(font
@@
 				)
 				(justify left top)
+			)
+		)
+		(pin "I2C_LP{I2C}" bidirectional
+			(at 227.33 64.77 180)
+			(effects
+				(font
+					(size 1.27 1.27)
+				)
+				(justify left)
 			)
 		)
@@
 			)
 		)
+		(pin "I2C_PD{I2C}" bidirectional
+			(at 227.33 119.38 180)
+			(effects
+				(font
+					(size 1.27 1.27)
+				)
+				(justify left)
+			)
+		)
+		(pin "I2C_LP{I2C}" bidirectional
+			(at 227.33 123.19 180)
+			(effects
+				(font
+					(size 1.27 1.27)
+				)
+				(justify left)
+			)
+		)
 		(instances
 			(project "Ducker-Charger"
@@
 	)
 	(sheet
-		(at 226.695 32.385)
+		(at 227.33 74.93)
 		(size 44.45 35.56)
 		(exclude_from_sim no)
@@
 		)
 		(property "Sheetname" "High_pow"
-			(at 226.695 31.6734 0)
+			(at 227.33 74.2184 0)
 			(effects
 				(font
@@
 		)
 		(property "Sheetfile" "high_pow.kicad_sch"
-			(at 226.695 68.5296 0)
+			(at 227.33 111.0746 0)
 			(effects
 				(font
@@
 			)
 		)
+		(pin "I2C_PD{I2C}" bidirectional
+			(at 227.33 106.68 180)
+			(effects
+				(font
+					(size 1.27 1.27)
+				)
+				(justify left)
+			)
+		)
