File: PCB/Ducker-Charger/Ducker-Charger.kicad_pcb (KiCad board)
At the start: 4 copper layers, 66.4 x 163.6 mm, 259 parts, among them CN401 100n, IC301 STUSB4710AQ1TR, IC401 TPS54202HDDCT, IC501 BQ34Z100PWR-R2, J101 Conn_01x02, J102 Conn_01x05, J301 USB_A, J302 USB_A, J303 Conn_01x02, J401 Debug, J403 Conn_01x08, J404 Conn_01x08, Q201 BSC040N08NS5, Q202 BSC040N08NS5, Q203 BSC040N08NS5, Q204 BSC040N08NS5, Q205 AO4407A, Q301 AO3400A, Q302 AO3400A, Q303 AO3400A, Q304 AO3400A, Q305 AO4407A, Q306 AO4407A, Q401 AO3400A, Q402 PMOS, Q501 BSC040N08NS5, Q502 BSC040N08NS5, Q503 BC846, SW401 EC11E15244G1, SW403 Reset, U201 BQ25713RSNR, U202 TPS25750DRJKR, U203 TPS54302, U301 INA3221, U302 STPD01PUR, U303 TPS54302, U304 TPS54302, U401 STM32F401RBT6, U501 BQ7791500PWR, U502 ISO1540DR, Y401 16MHz

Commit message: feat: final version before prod
Parts:
- removed F101: 3522-2, EasyEDA:FUSE-TH_3522-2
- removed the G*** at (176.7, 110.9)
- removed IC301: STUSB4710AQ1TR, Package_DFN_QFN:QFN-16-1EP_3x3mm_P0.5mm_EP1.7x1.7mm
- removed R317: 50, Resistor_SMD:R_0603_1608Metric
- added C247: 4.7u, Capacitor_SMD:C_0805_2012Metric, F.Cu at (104.1, 175.0)
- added C248: 4.7u, Capacitor_SMD:C_0805_2012Metric, F.Cu at (73.2, 177.2)
- added C249: 10n, Capacitor_SMD:C_0603_1608Metric, F.Cu at (75.1, 177.1)
- added C314: 1u, Resistor_SMD:R_0603_1608Metric, F.Cu at (116.3, 134.9)
- added C327: 2.2u, Capacitor_SMD:C_0805_2012Metric, F.Cu at (119.0, 132.9)
- added C391: 100n, Resistor_SMD:R_0603_1608Metric, F.Cu at (119.1, 134.7)
- added D302: LED, LED_SMD:LED_0603_1608Metric, F.Cu at (114.5, 139.7)
- added F102: 20A, Fuse:Fuseholder_Cylinder-5x20mm_Schurter_0031_8201_Horizontal_Open, F.Cu at (77.3, 31.1)
- added IC302: CYPD3175-24LQXQ, KiCad:QFN50P400X400X60-25N-D, F.Cu at (119.6, 138.3)
- added J304: Debug, Eagle_Connectors:SAMTEC_FTSH-107-01-L-DV-K-TR, B.Cu at (128.1, 146.0)
- added R318: 1k, Resistor_SMD:R_0603_1608Metric, F.Cu at (115.3, 137.5)
- added kibuzzard-6A3BBBB4: G***, kibuzzard-6A3BBBB4, F.Cu at (79.5, 85.4)
- added kibuzzard-6A3BBBD7: G***, kibuzzard-6A3BBBD7, F.Cu at (79.5, 98.1)
- added kibuzzard-6A3BBBE2: G***, kibuzzard-6A3BBBE2, F.Cu at (79.5, 109.2)
- added kibuzzard-6A3BBBEB: G***, kibuzzard-6A3BBBEB, F.Cu at (79.5, 120.3)
- added kibuzzard-6A3BBBFC: G***, kibuzzard-6A3BBBFC, F.Cu at (79.5, 140.2)
- added kibuzzard-6A3BBC07: G***, kibuzzard-6A3BBC07, F.Cu at (79.5, 144.2)
- added kibuzzard-6A3BBC42: G***, kibuzzard-6A3BBC42, F.Cu at (71.2, 40.8)
- added kibuzzard-6A3BBDB6: G***, kibuzzard-6A3BBDB6, F.Cu at (133.5, 86.5)
- added kibuzzard-6A3BBDBF: G***, kibuzzard-6A3BBDBF, F.Cu at (133.5, 104.4)
- added kibuzzard-6A3BBDD0: G***, kibuzzard-6A3BBDD0, F.Cu at (133.5, 129.8)
- added kibuzzard-6A3BBDD9: G***, kibuzzard-6A3BBDD9, F.Cu at (133.5, 149.9)
- added kibuzzard-6A3C421F: G***, kibuzzard-6A3C421F, F.Cu at (75.0, 186.9)
- C231: moved to B.Cu
- C305: value 1u -> 390p; footprint Capacitor_SMD:C_0805_2012Metric -> Resistor_SMD:R_0603_1608Metric
- C308: value 1u -> 390p; footprint Capacitor_SMD:C_0603_1608Metric -> Resistor_SMD:R_0603_1608Metric
- C309: value 1u -> 100n; footprint Capacitor_SMD:C_0805_2012Metric -> Resistor_SMD:R_0603_1608Metric
- R311: value 10 -> 200k
- R316: value 1k2 -> 63k
- moved G*** 180.9 mm to (129.0, 181.7)
- moved G*** 98.2 mm to (101.2, 99.8)
- moved kibuzzard-694FF1FC 94.3 mm to (99.4, 29.9)
- moved kibuzzard-694FF228 94.3 mm to (102.0, 29.9)
- moved kibuzzard-694FF21A 94.3 mm to (97.0, 29.9)
- moved kibuzzard-694FF236 94.3 mm to (104.7, 29.9)
- moved kibuzzard-694FF248 94.3 mm to (107.1, 29.9)
- moved R311 7.15 mm to (125.3, 133.9)
- moved C309 5.36 mm to (121.7, 133.9), turned to 90 degrees
- moved C305 5.01 mm to (123.1, 137.7), turned to 90 degrees
- moved C308 1.90 mm to (124.7, 138.5), turned to 90 degrees
- moved C237 1.52 mm to (72.9, 174.3)
- moved C238 1.52 mm to (72.9, 171.9)
- moved C235 1.52 mm to (72.9, 164.9)
- moved C236 1.52 mm to (72.9, 162.6)
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Connections:
- C305 pad 1: Net-(IC301-VREG_1V2) -> /Low_pow/CC1
- C308 pad 1: Net-(IC301-VDD) -> /Low_pow/CC2
- R311 pad 1: Net-(IC301-VDD) -> /Low_pow/VBUS
- R311 pad 2: +BATT -> Net-(IC302-FB)
- R316 pad 1: Net-(IC301-VBUS_SENSE) -> Net-(IC302-FB)
- R316 pad 2: /Low_pow/VBUS -> GND
Routing:
- net +BATT: track 103.1 -> 83.4 mm, vias 4 -> 332
- net /BMS/I2C_LP.SDA: track 223.6 -> 240.7 mm, vias 8 -> 7
- net GND: track 212.8 -> 229.2 mm, vias 175 -> 195
- net /Low_pow/~{RESET}: track 0.00 -> 16.4 mm, vias 0 -> 1
- net /Low_pow/SWCLK: track 0.00 -> 12.8 mm, vias 0 -> 1
- net /Low_pow/SWDIO: track 0.00 -> 12.3 mm, vias 0 -> 1
- net /Low_pow/VBUS: track 52.7 -> 64.4 mm, vias 9 -> 11
- net Net-(IC301-VBUS_DISCH): track 10.9 -> 0.00 mm, vias 2 -> 0
- net VSYS: track 228.1 -> 238.7 mm
- net /BMS/I2C_LP.SCL: track 233.8 -> 244.0 mm
- net Net-(IC301-VBUS_SENSE): track 9.30 -> 0.00 mm, vias 2 -> 0
- net +3V3: track 71.6 -> 77.8 mm, vias 34 -> 37
- net /Logic/C2.RDY: track 96.2 -> 90.4 mm
- net Net-(IC302-FB): track 0.00 -> 5.84 mm
- net Net-(IC301-VDD): track 4.84 -> 0.00 mm
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- added copper zone on In2.Cu, net /Low_pow/VBUS
Other:
- board text added: "*"
- board text added: "3V3"
- board text added: "<solder"
- board text added: "GND"
