File: PCB/Ducker-Charger/BMS.kicad_sch (KiCad schematic)
At the start: 44 parts, among them IC501 BQ34Z100PWR-R2, Q501 BSC040N08NS5, Q502 BSC040N08NS5, Q503 BC846, U501 BQ7791500PWR, U502 ISO1540DR

Commit message: feat: production BOM
Parts:
- C501, C502, C503, C504, C509, C_VDD501, C_VDD502: Manufacturer_Name (none) -> Samsung; Manufacturer_Part_Number (none) -> CL21B105KBFNNNG
- C505, C506, C507, C508: Manufacturer_Name (none) -> Samsung; Manufacturer_Part_Number (none) -> CL10B104KB8NNNC
- C510: Manufacturer_Name (none) -> TDK; Manufacturer_Part_Number (none) -> C2012X5R1E475K125AB
- D501: Manufacturer_Name (none) -> onsemi; Manufacturer_Part_Number (none) -> MMSZ5231BT1G
- Q501, Q502: Manufacturer_Name (none) -> Infineon; Manufacturer_Part_Number (none) -> BSC040N08NS5ATMA1
- Q503: Manufacturer_Name (none) -> onsemi; Manufacturer_Part_Number (none) -> BC846BLT1G
- R501: Manufacturer_Name (none) -> Yageo; Manufacturer_Part_Number (none) -> RC0603JR-070RL
- R502, R503, R504, R505, R506, RCHG501, RDSG501, R_VDD501: Manufacturer_Name (none) -> Yageo; Manufacturer_Part_Number (none) -> RC0603FR-071KL
- R507: Manufacturer_Name (none) -> Yageo; Manufacturer_Part_Number (none) -> RC0603FR-07100KL
- R508, R509: Manufacturer_Name (none) -> Yageo; Manufacturer_Part_Number (none) -> RC0603FR-07100RL
- R510, TH501, TH502: Manufacturer_Name (none) -> Yageo; Manufacturer_Part_Number (none) -> RC0603FR-0710KL
- R511: Manufacturer_Name (none) -> Yageo; Manufacturer_Part_Number (none) -> RC0603FR-07220KL
- R512: Manufacturer_Name (none) -> Yageo; Manufacturer_Part_Number (none) -> RC0603FR-07300KL
- R513: Manufacturer_Name (none) -> Yageo; Manufacturer_Part_Number (none) -> RC0603FR-0716K5L
- R514, R516: Manufacturer_Name (none) -> Yageo; Manufacturer_Part_Number (none) -> RC0603FR-074K7L
- R515: Manufacturer_Name (none) -> Yageo; Manufacturer_Part_Number (none) -> RC0603FR-0715KL
- RGS501, RGS502: Manufacturer_Name (none) -> Yageo; Manufacturer_Part_Number (none) -> RC0603FR-071ML
- RLD501: Manufacturer_Name (none) -> Panasonic; Manufacturer_Part_Number (none) -> ERJ-3EKF4703V
- RSNS501: Manufacturer_Name (none) -> Bourns; Manufacturer_Part_Number (none) -> CSS2H-3920K-2L00F
- U501: Manufacturer_Name (none) -> Texas Instruments; Manufacturer_Part_Number (none) -> BQ7791500PWR
- U502: Manufacturer_Name (none) -> Analog Devices; Manufacturer_Part_Number (none) -> ADUM1250ARZ
