File: PCB/Ducker-Charger/Logic.kicad_sch (KiCad schematic)
At the start: 60 parts, among them CN401 100n, IC401 TPS54202HDDCT, J401 Debug, J403 Conn_01x08, J404 Conn_01x08, Q401 AO3400A, Q402 PMOS, SW401 EC11E15244G1, SW403 Reset, U401 STM32F401RBT6, Y401 16MHz

Commit message: feat: production BOM
Parts:
- C401, C402, C403, C405, C406, C407, C410, C411, C415, C420, CVBAT401: Manufacturer_Name (none) -> Samsung; Manufacturer_Part_Number (none) -> CL10B104KB8NNNC
- C404: Manufacturer_Name (none) -> Samsung; Manufacturer_Part_Number (none) -> CL21B105KBFNNNG
- C408: Manufacturer_Name (none) -> TDK; Manufacturer_Part_Number (none) -> C2012X5R1E225K125AC
- C409, C412: Manufacturer_Name (none) -> Murata; Manufacturer_Part_Number (none) -> GRM1885C1H180JA01D
- C413: Manufacturer_Name (none) -> Samsung; Manufacturer_Part_Number (none) -> CL31B106KBHNNNE
- C414, C416: Manufacturer_Name (none) -> Yageo; Manufacturer_Part_Number (none) -> CC0805KRX7R9BB104
- C417, C418: Manufacturer_Name (none) -> TDK; Manufacturer_Part_Number (none) -> C2012X5R1E226M125AC
- C419: Manufacturer_Name (none) -> KEMET; Manufacturer_Part_Number (none) -> C0805C750J5GACTU
- CN401: Manufacturer_Name (none) -> Kyocera AVX; Manufacturer_Part_Number (none) -> W3A43C104KAT2A
- D401: Manufacturer_Name (none) -> Bivar; Manufacturer_Part_Number (none) -> SM0603RC
- FB401: Manufacturer_Name (none) -> Murata; Manufacturer_Part_Number (none) -> BLM18KG601SN1D
- J401: Manufacturer_Name (none) -> Samtec; Manufacturer_Part_Number (none) -> FTSH-107-01-L-DV-K
- J403: Manufacturer_Name (none) -> Molex; Manufacturer_Part_Number (none) -> 200528-0080
- J404: Manufacturer_Name (none) -> JST; Manufacturer_Part_Number (none) -> B8B-EH-A(LF)(SN)
- L401: Manufacturer_Name (none) -> Bourns; Manufacturer_Part_Number (none) -> SRP6030VA-100M
- Q401: Manufacturer_Name (none) -> Alpha & Omega; Manufacturer_Part_Number (none) -> AO3400A
- Q402: Manufacturer_Name (none) -> Alpha & Omega; Manufacturer_Part_Number (none) -> AO3401A
- R401, R403, R404, R407, R415, R417, R419: Manufacturer_Name (none) -> Yageo; Manufacturer_Part_Number (none) -> RC0603FR-0710KL
- R402: Manufacturer_Name (none) -> Yageo; Manufacturer_Part_Number (none) -> RC0603FR-07220RL
- R405: Manufacturer_Name (none) -> Yageo; Manufacturer_Part_Number (none) -> RC0603FR-07511KL
- R406: Manufacturer_Name (none) -> Yageo; Manufacturer_Part_Number (none) -> RC0603FR-07105KL
- R408, R416, R418: Manufacturer_Name (none) -> Yageo; Manufacturer_Part_Number (none) -> RC0603FR-071KL
- R409, R410, R411, R412, R420: Manufacturer_Name (none) -> Yageo; Manufacturer_Part_Number (none) -> RC0603FR-074K7L
- R413: Manufacturer_Name (none) -> Yageo; Manufacturer_Part_Number (none) -> RC0603FR-0722K1L
- R414: Manufacturer_Name (none) -> Yageo; Manufacturer_Part_Number (none) -> RC0603FR-074K87L
- RN401: Manufacturer_Name (none) -> Yageo; Manufacturer_Part_Number (none) -> YC164-JR-0710KL
- SW403: Manufacturer_Name (none) -> TE Connectivity; Manufacturer_Part_Number (none) -> FSMSMTR
- U401: Manufacturer_Name (none) -> STMicroelectronics; Manufacturer_Part_Number (none) -> STM32F401RBT6
