File: PCB/Ducker-Charger/low_pow.kicad_sch (KiCad schematic)
At the start: 65 parts, among them IC302 CYPD3175-24LQXQ, J301 USB_A, J302 USB_A, J303 Conn_01x02, J304 Debug, Q301 AO3400A, Q302 AO3400A, Q303 AO3400A, Q304 AO3400A, Q305 AO4407A, Q306 AO4407A, U301 INA3221, U302 STPD01PUR, U303 TPS54302, U304 TPS54302

Commit message: feat: production BOM
Parts:
- C301, C302: Manufacturer_Name (none) -> Murata; Manufacturer_Part_Number (none) -> GRM21BR61H475KE51L
- C303, C304: Manufacturer_Name (none) -> Samsung; Manufacturer_Part_Number (none) -> CL31B106KBHNNNE
- C305, C308: Manufacturer_Name (none) -> Murata; Manufacturer_Part_Number (none) -> GRM1885C1H391JA01D
- C306, C307, C309, C391, CBOOT301: Manufacturer_Name (none) -> Samsung; Manufacturer_Part_Number (none) -> CL10B104KB8NNNC
- C310, C311, C312, C313: Manufacturer_Name (none) -> TDK; Manufacturer_Part_Number (none) -> C2012X5R1E226M125AC
- C314: Manufacturer_Name (none) -> Yageo; Manufacturer_Part_Number (none) -> CC0603KRX7R8BB105
- C327: Manufacturer_Name (none) -> TDK; Manufacturer_Part_Number (none) -> C2012X5R1E225K125AC
- CCDC301: Manufacturer_Name (none) -> Yageo; Manufacturer_Part_Number (none) -> CC0805KRX7R9BB472
- D301: Manufacturer_Name (none) -> STMicroelectronics; Manufacturer_Part_Number (none) -> USBLC6-2SC6
- D302: Manufacturer_Name (none) -> Bivar; Manufacturer_Part_Number (none) -> SM0603RC
- J301, J302: Manufacturer_Name (none) -> Molex; Manufacturer_Part_Number (none) -> 0676433910
- J303: Manufacturer_Name (none) -> TE Connectivity; Manufacturer_Part_Number (none) -> 282836-2
- J304: Manufacturer_Name (none) -> Samtec; Manufacturer_Part_Number (none) -> FTSH-107-01-L-DV-K
- L301, L302, L303: Manufacturer_Name (none) -> Bourns; Manufacturer_Part_Number (none) -> SRP7050TA-100M
- Q301, Q302, Q303, Q304: Manufacturer_Name (none) -> Alpha & Omega; Manufacturer_Part_Number (none) -> AO3400A
- Q305, Q306: Manufacturer_Name (none) -> Alpha & Omega; Manufacturer_Part_Number (none) -> AO4407A
- R301, R302, R318: Manufacturer_Name (none) -> Yageo; Manufacturer_Part_Number (none) -> RC0603FR-071KL
- R303, R304, R307, R308, R312, R314, Ron301: Manufacturer_Name (none) -> Yageo; Manufacturer_Part_Number (none) -> RC0603FR-07100KL
- R305, R306, R309, R310, RCDC301: Manufacturer_Name (none) -> Yageo; Manufacturer_Part_Number (none) -> RC0603FR-0710KL
- R311: Manufacturer_Name (none) -> Yageo; Manufacturer_Part_Number (none) -> RC0603FR-07200KL
- R313, R315: Manufacturer_Name (none) -> Yageo; Manufacturer_Part_Number (none) -> RC0603FR-0713K3L
- R316: Manufacturer_Name (none) -> Yageo; Manufacturer_Part_Number (none) -> RC0603FR-0762KL
- RCDC302: Manufacturer_Name (none) -> Yageo; Manufacturer_Part_Number (none) -> RC0603FR-075K6L
- U301: Manufacturer_Name (none) -> Texas Instruments; Manufacturer_Part_Number (none) -> INA3221AIRGVR
- U302: Manufacturer_Name (none) -> STMicroelectronics; Manufacturer_Part_Number (none) -> STPD01PUR
- U303, U304: Manufacturer_Name (none) -> Texas Instruments; Manufacturer_Part_Number (none) -> TPS54302DDCR
- USBC301: Manufacturer_Name (none) -> Same Sky; Manufacturer_Part_Number (none) -> UJ20-C-H-G-SMT-2A-P16-TR
