File: PCB/Sensing-Board/Sensing-Board.kicad_sch (KiCad schematic)
At the start: 0 parts

Commit message: feat: completed Sensing board
Parts:
- added J403: Conn_01x08, Connector_FFC-FPC:Molex_200528-0080_1x08-1MP_P1.00mm_Horizontal, symbol Connector_Generic:Conn_01x08
- added TH402, TH403, TH404, TH405: Thermistor_NTC, Resistor_SMD:R_0603_1608Metric, symbol Device:Thermistor_NTC
Connections:
- new net +3.3VA: J403.8 (Pin_8)
- new net GNDA: J403.7 (Pin_7), TH402.2, TH403.2, TH404.2, TH405.2
- new net NTC_1: J403.4 (Pin_4), TH402.1
- new net NTC_2: J403.3 (Pin_3), TH403.1
- new net NTC_3: J403.2 (Pin_2), TH404.1
- new net NTC_4: J403.1 (Pin_1), TH405.1
- no-connect marks 0 -> 2
